File: hardware/feather-mb-isa/isa.sch (EAGLE design)
At the start: 14 parts, among them J1 EDGE-80PTH-RA, J2 M22PTH, J3 GREEN-3P-5.0, J4 GREEN-3P-5.0, J5 GREEN-3P-5.0, J6 GREEN-3P-5.0

Commit message: Renamed midi.py
Now can be main.

Updated hardware. Looks ready for layout. Need to do some more
work in the middle. What to do with that space? Some neopixels?

Some buttons?

More headers?
Parts:
- added J12: (no value), SparkFun-Connectors:CONN_03
- added J19, J20, J21, J22, J23, J24, J25: (no value), SparkFun-Connectors:CONN_023.5MM
- added J7, J8: GREEN-3P-5.0, Seeed-Connector:SCREW-TERMINAL-GREEN(3P-5.0)
Connections:
- removed net 19: J1.A8, J2.21
- removed net 20: J1.A7, J2.22
- removed net M0RX: J2.16
- removed net M0TX: J2.12
- new net 3V: J12.2, MS1.3V
- new net D10: J22.2, MS1.GPIO10
- new net D11: J23.2, MS1.GPIO11
- new net D12: J24.2, MS1.GPIO12
- new net D13: J25.2, MS1.GPIO13
- new net D5: J19.2, MS1.GPIO5
- new net D6: J20.2, MS1.GPIO6
- new net D9: J21.2, MS1.GPIO9
- new net M4A0: J3.P$2, MS1.GPIOA0
- new net M4A1: J4.P$2, MS1.GPIOA1
- new net M4A2: J5.P$2, MS1.GPIOA2
- new net M4A3: J6.P$2, MS1.GPIOA3
- new net M4A4: J7.P$2, MS1.GPIOA4
- new net M4A5: J8.P$2, MS1.GPIOA5
- new net M4RX: J2.12, MS1.GPIORX
- new net M4TX: J2.16, MS1.GPIOTX
- new net MB3V: J12.1, J2.3
- new net SCL: J1.A8, J2.21, MS1.GPIOSCL
- new net SDA: J1.A7, J2.22, MS1.GPIOSDA
- net 10: no longer J6.P$2
- net 2: no longer J3.P$2
- net 3: no longer J4.P$2
- net 3.3V: now also J7.P$1, J8.P$1; no longer J2.3
- net 4: no longer J5.P$2
- net GND: now also J19.1, J20.1, J21.1, J22.1, J23.1, J24.1, J25.1, J7.P$3, J8.P$3, MS1.GND

Commit message: Changes.
Parts:
- added J10: (no value), SparkFun-Connectors:CONN_16LOCK
- added J11: (no value), SparkFun-Connectors:CONN_03SCREW
- added J9: (no value), SparkFun-Connectors:CONN_12LOCK
- added MS2: FEATHERWING_NODIM, adafruit:FEATHERWING_NODIM
- added U$3: LYNX#CORO#UNUM#PNG, lynx#coro#unum#png:LYNX#CORO#UNUM#PNG
- added U$4: LYNX#CORO#UNUM#PNG, big-lynx:LYNX#CORO#UNUM#PNG
Connections:
- removed net 3V: J12.2, MS1.3V
- new net AREF: J10.3, MS1.AREF, MS2.AREF
- new net EN: J9.11, MS1.EN, MS2.EN
- new net N$15: J10.16, MS2.NC
- new net QOWI: J10.12, MS1.GPIOMOSI, MS2.GPIOMOSI
- new net RESET: J10.1, MS1.!RESET, MS2.!RESET
- new net SCK: J10.11, MS1.GPIOSCK, MS2.GPIOSCK
- new net USB: J9.10, MS1.USB, MS2.USB
- new net VBAT: J9.12, MS1.VBAT, MS2.VBAT
- new net WOQI: J10.13, MS1.GPIOMISO, MS2.GPIOMISO
- net 3.3V: now also J10.2, J11.3, J12.2, MS1.3V, MS2.3V; no longer J1.A10, J1.A11, J1.A12, J1.A13, J1.A14, J1.A9
- net D10: now also J9.6, MS2.GPIO10
- net D11: now also J9.7, MS2.GPIO11
- net D12: now also J9.8, MS2.GPIO12
- net D13: now also J9.9, MS2.GPIO13
- net D5: now also J11.2, J9.3, MS2.GPIO5
- net D6: now also J9.4, MS2.GPIO6
- net D9: now also J9.5, MS2.GPIO9
- net GND: now also J10.4, J11.1, MS2.GND
- net M4A0: now also J10.5, MS2.GPIOA0
- net M4A1: now also J10.6, MS2.GPIOA1
- net M4A2: now also J10.7, MS2.GPIOA2
- net M4A3: now also J10.8, MS2.GPIOA3
- net M4A4: now also J10.9, MS2.GPIOA4
- net M4A5: now also J10.10, MS2.GPIOA5
- net M4RX: now also J10.14, MS2.GPIORX
- net M4TX: now also J10.15, MS2.GPIOTX
- net MB3V: now also J1.A10, J1.A11, J1.A12, J1.A13, J1.A14, J1.A9
- net SCL: now also J9.2, MS2.GPIOSCL
- net SDA: now also J9.1, MS2.GPIOSDA

Commit message: Updates to the board.
It would be good to have one pin with power. The ids are all out of order on the RH side.
Parts:
- removed J25: (no value), SparkFun-Connectors:CONN_023.5MM
Connections:
- net D13: no longer J25.2
- net GND: no longer J25.1
Changed lines of the file:
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@@
 <part name="J23" library="SparkFun-Connectors" library_urn="urn:adsk.eagle:library:513" deviceset="CONN_02" device="3.5MM" package3d_urn="urn:adsk.eagle:package:38050/1"/>
 <part name="J24" library="SparkFun-Connectors" library_urn="urn:adsk.eagle:library:513" deviceset="CONN_02" device="3.5MM" package3d_urn="urn:adsk.eagle:package:38050/1"/>
-<part name="J25" library="SparkFun-Connectors" library_urn="urn:adsk.eagle:library:513" deviceset="CONN_02" device="3.5MM" package3d_urn="urn:adsk.eagle:package:38050/1"/>
 <part name="GND12" library="SparkFun-PowerSymbols" library_urn="urn:adsk.eagle:library:530" deviceset="GND" device=""/>
 <part name="GND13" library="SparkFun-PowerSymbols" library_urn="urn:adsk.eagle:library:530" deviceset="GND" device=""/>
@@
 <attribute name="NAME" x="325.12" y="69.088" size="1.778" layer="95" font="vector"/>
 </instance>
-<instance part="J25" gate="G$1" x="327.66" y="48.26" smashed="yes">
-<attribute name="VALUE" x="325.12" y="43.434" size="1.778" layer="96" font="vector"/>
-<attribute name="NAME" x="325.12" y="53.848" size="1.778" layer="95" font="vector"/>
-</instance>
 <instance part="GND12" gate="1" x="302.26" y="12.7" smashed="yes">
 <attribute name="VALUE" x="302.26" y="12.446" size="1.778" layer="96" align="top-center"/>
@@
 <pinref part="GND13" gate="1" pin="GND"/>
 <wire x1="337.82" y1="63.5" x2="337.82" y2="48.26" width="0.1524" layer="91"/>
-<pinref part="J25" gate="G$1" pin="1"/>
 <wire x1="337.82" y1="48.26" x2="337.82" y2="40.64" width="0.1524" layer="91"/>
 <wire x1="335.28" y1="48.26" x2="337.82" y2="48.26" width="0.1524" layer="91"/>
@@
 </segment>
 <segment>
-<pinref part="J25" gate="G$1" pin="2"/>
 <wire x1="335.28" y1="50.8" x2="342.9" y2="50.8" width="0.1524" layer="91"/>
 <label x="342.9" y="50.8" size="1.016" layer="95" xref="yes"/>

Commit message: Moving things around.
Parts:
- J3, J4, J5, J6, J7, J8: value GREEN-3P-5.0 -> (none); device Seeed-Connector:SCREW-TERMINAL-GREEN(3P-5.0) -> SparkFun-Connectors:CONN_03SCREW
Connections:
- removed net 12: J1.A23
- removed net 8: J1.A27
- net 3.3V: now also J3.1, J4.1, J5.1, J6.1, J7.1, J8.1; no longer J3.P$1, J4.P$1, J5.P$1, J6.P$1, J7.P$1, J8.P$1
- net D13: now also J11.2
- net D5: no longer J11.2
- net GND: now also J3.3, J4.3, J5.3, J6.3, J7.3, J8.3; no longer J3.P$3, J4.P$3, J5.P$3, J6.P$3, J7.P$3, J8.P$3
- net M4A0: now also J3.2; no longer J3.P$2
- net M4A1: now also J4.2; no longer J4.P$2
- net M4A2: now also J5.2; no longer J5.P$2
- net M4A3: now also J8.2; no longer J6.P$2
- net M4A4: now also J6.2; no longer J7.P$2
- net M4A5: now also J7.2; no longer J8.P$2
- net M4RX: now also J1.A27
- net M4TX: now also J1.A23
Other:
- moved on the sheet: J11
